File: 2-Power.kicad_sch (KiCad schematic)
At the start: 15 parts, among them J201 Molex PicoBlade, U201 ZXMP3A17E6TA

Commit message: Schematic: improving comments about ESD protection
Other:
- note added: "TVS diode: - bidirectional because it's followed by reverse polarity protection - also protects from high inputs applied when battery is off, leaking through opamp inputs - reverse standoff 20V, breakdown 21-25V, clamping 27-30V"
- note removed: "TVS diode: - bidirectional because it's followed by reverse polarity protection - also protects from high inputs applied when battery is off, leaking through opamp inputs - reverse standoff 20V, clamping"
Changed lines of the file:
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@@
     (effects (font (size 1 1)) (justify left bottom))
   )
-  (text "TVS diode:\n- bidirectional because it's followed \nby reverse polarity protection \n- also protects from high inputs applied \nwhen battery is off, leaking through \nopamp inputs\n- reverse standoff 20V, clamping "
-    (at 94.615 43.18 0)
+  (text "TVS diode:\n- bidirectional because it's followed \nby reverse polarity protection \n- also protects from high inputs applied \nwhen battery is off, leaking through \nopamp inputs\n- reverse standoff 20V, breakdown 21-25V,\nclamping 27-30V"
+    (at 92.71 43.815 0)
     (effects (font (size 1 1)) (justify left bottom))
   )

Commit message: correcting the filter name to HPF in schematic, board and in exported schematics
Parts:
- gave numbers to parts that had none: 7
- renumbered C5 to C204, C5 to C205, C5 to C206, C5 to C207, D1 to D201
