File: 2-Power.kicad_sch (KiCad schematic)
At the start: 17 parts, among them J201 DC IN 5.5/2.1mm, J202 9V Battery Connector, U201 ZXMP3A17E6TA

Commit message: schematic: finishing standoffs, screws, minor improvements
Parts:
- J202: now left out of the parts list
- S201: Source Mouser -> TME
Changed lines of the file:
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@@
 		)
 		(instances
-			(project "2023_PiezoPreamp"
+			(project "2024_PiezoPreamp3"
 				(path "/6e141482-2809-49ad-b316-4cdedc98ad26/b10e95cd-10a1-4d25-b6a0-2bd4304f390c"
 					(reference "#PWR018")
@@
 		)
 		(instances
-			(project "2023_PiezoPreamp"
+			(project "2024_PiezoPreamp3"
 				(path "/6e141482-2809-49ad-b316-4cdedc98ad26/b10e95cd-10a1-4d25-b6a0-2bd4304f390c"
 					(reference "#PWR028")
@@
 		)
 		(instances
-			(project "2023_PiezoPreamp"
+			(project "2024_PiezoPreamp3"
 				(path "/6e141482-2809-49ad-b316-4cdedc98ad26/b10e95cd-10a1-4d25-b6a0-2bd4304f390c"
 					(reference "#FLG02")
@@
 		)
 		(instances
-			(project "2023_PiezoPreamp"
+			(project "2024_PiezoPreamp3"
 				(path "/6e141482-2809-49ad-b316-4cdedc98ad26/b10e95cd-10a1-4d25-b6a0-2bd4304f390c"
 					(reference "#FLG01")
@@
 			)
 		)
-		(property "Source" "Mouser"
+		(property "Source" "TME"
 			(at 49.53 121.92 0)
 			(effects
@@
 		)
 		(instances
-			(project "2023_PiezoPreamp"
+			(project "2024_PiezoPreamp3"
 				(path "/6e141482-2809-49ad-b316-4cdedc98ad26/b10e95cd-10a1-4d25-b6a0-2bd4304f390c"
 					(reference "S201")
@@
 		)
 		(instances
-			(project "2023_PiezoPreamp"
+			(project "2024_PiezoPreamp3"
 				(path "/6e141482-2809-49ad-b316-4cdedc98ad26/b10e95cd-10a1-4d25-b6a0-2bd4304f390c"
 					(reference "#PWR015")
@@
 		)
 		(instances
-			(project "2023_PiezoPreamp"
+			(project "2024_PiezoPreamp3"
 				(path "/6e141482-2809-49ad-b316-4cdedc98ad26/b10e95cd-10a1-4d25-b6a0-2bd4304f390c"
 					(reference "C203")
@@
 		)
 		(instances
-			(project "2023_PiezoPreamp"
+			(project "2024_PiezoPreamp3"
 				(path "/6e141482-2809-49ad-b316-4cdedc98ad26/b10e95cd-10a1-4d25-b6a0-2bd4304f390c"
 					(reference "C202")
@@
 		)
 		(instances
-			(project "2023_PiezoPreamp"
+			(project "2024_PiezoPreamp3"
 				(path "/6e141482-2809-49ad-b316-4cdedc98ad26/b10e95cd-10a1-4d25-b6a0-2bd4304f390c"
 					(reference "R201")
@@
 		)
 		(instances
-			(project "2023_PiezoPreamp"
+			(project "2024_PiezoPreamp3"
 				(path "/6e141482-2809-49ad-b316-4cdedc98ad26/b10e95cd-10a1-4d25-b6a0-2bd4304f390c"
 					(reference "#PWR02")
@@
 		)
 		(instances
-			(project "2023_PiezoPreamp"
+			(project "2024_PiezoPreamp3"
 				(path "/6e141482-2809-49ad-b316-4cdedc98ad26/b10e95cd-10a1-4d25-b6a0-2bd4304f390c"
 					(reference "C201")
@@
 		)
 		(instances
-			(project "2023_PiezoPreamp"
+			(project "2024_PiezoPreamp3"
 				(path "/6e141482-2809-49ad-b316-4cdedc98ad26/b10e95cd-10a1-4d25-b6a0-2bd4304f390c"
 					(reference "R202")
@@
 		)
 		(instances
-			(project "2023_PiezoPreamp"
+			(project "2024_PiezoPreamp3"
 				(path "/6e141482-2809-49ad-b316-4cdedc98ad26/b10e95cd-10a1-4d25-b6a0-2bd4304f390c"
 					(reference "#PWR029")
@@
 		)
 		(instances
-			(project "2023_PiezoPreamp"
+			(project "2024_PiezoPreamp3"
 				(path "/6e141482-2809-49ad-b316-4cdedc98ad26/b10e95cd-10a1-4d25-b6a0-2bd4304f390c"
 					(reference "#PWR01")
@@
 		)
 		(instances
-			(project "2023_PiezoPreamp"
+			(project "2024_PiezoPreamp3"
 				(path "/6e141482-2809-49ad-b316-4cdedc98ad26/b10e95cd-10a1-4d25-b6a0-2bd4304f390c"
 					(reference "R203")
@@
 		(unit 1)
 		(exclude_from_sim no)
-		(in_bom yes)
-		(on_board yes)
+		(in_bom no)
+		(on_board no)
 		(dnp no)
 		(property "Reference" "J202"
@@
 		)
 		(instances
-			(project "2023_PiezoPreamp"
+			(project "2024_PiezoPreamp3"
 				(path "/6e141482-2809-49ad-b316-4cdedc98ad26/b10e95cd-10a1-4d25-b6a0-2bd4304f390c"
 					(reference "J202")
@@
 		)
 		(instances
-			(project "2023_PiezoPreamp"
+			(project "2024_PiezoPreamp3"
 				(path "/6e141482-2809-49ad-b316-4cdedc98ad26/b10e95cd-10a1-4d25-b6a0-2bd4304f390c"
 					(reference "C207")
@@
 		)
 		(instances
-			(project "2023_PiezoPreamp"
+			(project "2024_PiezoPreamp3"
 				(path "/6e141482-2809-49ad-b316-4cdedc98ad26/b10e95cd-10a1-4d25-b6a0-2bd4304f390c"
 					(reference "U201")
@@
 		)
 		(instances
-			(project "2023_PiezoPreamp"
+			(project "2024_PiezoPreamp3"
 				(path "/6e141482-2809-49ad-b316-4cdedc98ad26/b10e95cd-10a1-4d25-b6a0-2bd4304f390c"
 					(reference "#PWR014")
@@
 		)
 		(instances
-			(project "2023_PiezoPreamp"
+			(project "2024_PiezoPreamp3"
 				(path "/6e141482-2809-49ad-b316-4cdedc98ad26/b10e95cd-10a1-4d25-b6a0-2bd4304f390c"
 					(reference "#PWR04")
@@
 		)
 		(instances
-			(project "2023_PiezoPreamp"
+			(project "2024_PiezoPreamp3"
 				(path "/6e141482-2809-49ad-b316-4cdedc98ad26/b10e95cd-10a1-4d25-b6a0-2bd4304f390c"
 					(reference "J201")
@@
 		)
 		(instances
-			(project "2023_PiezoPreamp"
+			(project "2024_PiezoPreamp3"
 				(path "/6e141482-2809-49ad-b316-4cdedc98ad26/b10e95cd-10a1-4d25-b6a0-2bd4304f390c"
 					(reference "R204")
@@
 		)
 		(instances
-			(project "2023_PiezoPreamp"
+			(project "2024_PiezoPreamp3"
 				(path "/6e141482-2809-49ad-b316-4cdedc98ad26/b10e95cd-10a1-4d25-b6a0-2bd4304f390c"
 					(reference "#PWR06")
@@
 		)
 		(instances
-			(project "2023_PiezoPreamp"
+			(project "2024_PiezoPreamp3"
 				(path "/6e141482-2809-49ad-b316-4cdedc98ad26/b10e95cd-10a1-4d25-b6a0-2bd4304f390c"
 					(reference "C204")
@@
 		)
 		(instances
-			(project "2023_PiezoPreamp"
+			(project "2024_PiezoPreamp3"
 				(path "/6e141482-2809-49ad-b316-4cdedc98ad26/b10e95cd-10a1-4d25-b6a0-2bd4304f390c"
 					(reference "C205")
@@
 		)
 		(instances
-			(project "2023_PiezoPreamp"
+			(project "2024_PiezoPreamp3"
 				(path "/6e141482-2809-49ad-b316-4cdedc98ad26/b10e95cd-10a1-4d25-b6a0-2bd4304f390c"
 					(reference "C206")
@@
 		)
 		(instances
-			(project "2023_PiezoPreamp"
+			(project "2024_PiezoPreamp3"
 				(path "/6e141482-2809-49ad-b316-4cdedc98ad26/b10e95cd-10a1-4d25-b6a0-2bd4304f390c"
 					(reference "D202")
@@
 		)
 		(instances
-			(project "2023_PiezoPreamp"
+			(project "2024_PiezoPreamp3"
 				(path "/6e141482-2809-49ad-b316-4cdedc98ad26/b10e95cd-10a1-4d25-b6a0-2bd4304f390c"
 					(reference "D201")
@@
 		)
 		(instances
-			(project "2023_PiezoPreamp"
+			(project "2024_PiezoPreamp3"
 				(path "/6e141482-2809-49ad-b316-4cdedc98ad26/b10e95cd-10a1-4d25-b6a0-2bd4304f390c"
 					(reference "#PWR010")
@@
 		)
 		(instances
-			(project "2023_PiezoPreamp"
+			(project "2024_PiezoPreamp3"
 				(path "/6e141482-2809-49ad-b316-4cdedc98ad26/b10e95cd-10a1-4d25-b6a0-2bd4304f390c"
 					(reference "#PWR016")
@@
 		)
 		(instances
-			(project "2023_PiezoPreamp"
+			(project "2024_PiezoPreamp3"
 				(path "/6e141482-2809-49ad-b316-4cdedc98ad26/b10e95cd-10a1-4d25-b6a0-2bd4304f390c"
 					(reference "#PWR017")
@@
 		)
 		(instances
-			(project "2023_PiezoPreamp"
+			(project "2024_PiezoPreamp3"
 				(path "/6e141482-2809-49ad-b316-4cdedc98ad26/b10e95cd-10a1-4d25-b6a0-2bd4304f390c"
 					(reference "#PWR08")
@@
 		)
 		(instances
-			(project "2023_PiezoPreamp"
+			(project "2024_PiezoPreamp3"
 				(path "/6e141482-2809-49ad-b316-4cdedc98ad26/b10e95cd-10a1-4d25-b6a0-2bd4304f390c"
 					(reference "#PWR07")
