File: 1-ChargeAmpAndEQ.kicad_sch (KiCad schematic)
At the start: 58 parts, among them J101 6.3mm stereo, J102 6.3mm stereo, U101 OPA145, U102 OPA145

Commit message: schematic: optimizing few BOM items (for less costly alternatives), few updates
Parts:
- Cb103, Chp107: footprint library:GRM31C5C2A104JA01L -> library:GRM31C5C1H104JA01L; Alt (none) -> GRM31C5C2A104JA01L; LCSC Part # C405303 -> C97946; Mfr Part # GRM31C5C2A104JA01L -> GRM31C5C1H104JA01L; Mouser Part # 81-GRM31C5C2A104JA1L -> 81-GRM31C5C1H104JA1L; TME Part # (none) -> -
- H101, H104, H107: footprint library:FreePad_1.1mm_2.0mm -> library:FreePad_1.1mm_2.1mm_rect
- H102, H103, H105, H106, H108, H109: footprint library:FreePad_1.1mm_2.0mm -> library:FreePad_1.1mm_2.1mm
- R101, R102: footprint library:RT0603BRE07150RL_UL-M -> library:ERA-3AEB151V; Alt (none) -> RT0603BRE07150RL; LCSC Part # C728601 -> C543626; Mfr Yageo -> Panasonic; Mfr Part # RT0603BRE07150RL -> ERA3AEB151V; Mouser Part # 603-RT0603BRE07150RL -> 667-ERA-3AEB151V; TME Part # (none) -> -
- R103, Rb101, Rb102: footprint library:ERA-3AEB392V -> library:RT0603FRE073K9L; Alt (none) -> ERA-3AEB392V; LCSC Part # C473237 -> C863790; Mfr Panasonic -> Yageo; Mfr Part # ERA-3AEB392V -> RT0603FRE073K9L; Mouser Part # 667-ERA-3AEB392V -> 603-RT0603FRE073K9L; TME Part # (none) -> -
- S101, S102: Alt (none) -> SK14D01G6L
- U101, U102: Alt (none) -> OP2134

Commit message: schematic, PCB: many small adjustments before fab&assembly
Parts:
- U101, U102: JLCPCB Rotation Offset (none) -> 180
