File: 3-BatteryIndicator.kicad_sch (KiCad schematic)
At the start: 11 parts, among them U301 BC847BS,115

Commit message: schematic: optimizing few BOM items (for less costly alternatives), few updates
Parts:
- D301: Alt (none) -> APTD1608LSURCK same footprint
- R301, R302, R304: footprint library:RT0603BRD0747KL -> library:RT0603FRD0747KL; Alt (none) -> RT0603BRD0747KL; LCSC Part # C326725 -> C728633; Mfr Part # RT0603BRD0747KL -> RT0603FRD0747KL; Mouser Part # 603-RT0603BRD0747KL -> 603-RT0603FRD0747KL; TME Part # (none) -> -
- R303: footprint library:ERA-3AEB392V -> library:RT0603FRE073K9L; Alt (none) -> ERA-3AEB392V; LCSC Part # C473237 -> C863790; Mfr Panasonic -> Yageo; Mfr Part # ERA-3AEB392V -> RT0603FRE073K9L; Mouser Part # 667-ERA-3AEB392V -> 603-RT0603FRE073K9L; TME Part # (none) -> -
- S301: Alt (none) -> OS102011MA1QN1C, OS102011MA1QS1, OS102011MA1QS1C, 1825232-1
Changed lines of the file:
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@@
 	(title_block
 		(title "Battery & Power Indicator")
-		(date "2024-03-07")
+		(date "2024-03-10")
 		(rev "3.0")
 		(company "Arx")
@@
 		)
 		(property "Source" "LCSC"
+			(at 219.71 60.96 0)
+			(effects
+				(font
+					(size 1.27 1.27)
+				)
+				(hide yes)
+			)
+		)
+		(property "Alt" "APTD1608LSURCK same footprint"
 			(at 219.71 60.96 0)
 			(effects
@@
 			)
 		)
-		(property "Footprint" "library:RT0603BRD0747KL"
+		(property "Footprint" "library:RT0603FRD0747KL"
 			(at 90.17 71.12 0)
 			(effects
@@
 			)
 		)
-		(property "LCSC Part #" "C326725"
+		(property "LCSC Part #" "C728633"
 			(at 90.17 71.12 0)
 			(effects
@@
 			)
 		)
-		(property "Mfr Part #" "RT0603BRD0747KL"
+		(property "Mfr Part #" "RT0603FRD0747KL"
 			(at 90.17 71.12 0)
 			(effects
@@
 			)
 		)
-		(property "Mouser Part #" "603-RT0603BRD0747KL"
+		(property "Mouser Part #" "603-RT0603FRD0747KL "
 			(at 90.17 71.12 0)
 			(effects
@@
 		)
 		(property "Source" "LCSC"
+			(at 90.17 71.12 0)
+			(effects
+				(font
+					(size 1.27 1.27)
+				)
+				(hide yes)
+			)
+		)
+		(property "Alt" "RT0603BRD0747KL"
+			(at 90.17 71.12 0)
+			(effects
+				(font
+					(size 1.27 1.27)
+				)
+				(hide yes)
+			)
+		)
+		(property "TME Part #" "-"
 			(at 90.17 71.12 0)
 			(effects
@@
 			)
 		)
-		(property "Footprint" "library:ERA-3AEB392V"
+		(property "Footprint" "library:RT0603FRE073K9L"
 			(at 90.17 95.25 0)
 			(effects
@@
 			)
 		)
-		(property "Datasheet" "https://cz.mouser.com/datasheet/2/315/AOA0000C307-1149632.pdf"
+		(property "Datasheet" "https://cz.mouser.com/datasheet/2/447/PYu_RT_1_to_0_01_RoHS_L_12-3003070.pdf"
 			(at 90.17 95.25 0)
 			(effects
@@
 			)
 		)
-		(property "Mfr" "Panasonic"
+		(property "Mfr" "Yageo"
 			(at 90.17 95.25 0)
 			(effects
@@
 			)
 		)
-		(property "Mfr Part #" "ERA-3AEB392V"
+		(property "Mfr Part #" "RT0603FRE073K9L"
 			(at 90.17 95.25 0)
 			(effects
@@
 			)
 		)
-		(property "Mouser Part #" "667-ERA-3AEB392V"
+		(property "Mouser Part #" "603-RT0603FRE073K9L "
 			(at 90.17 95.25 0)
 			(effects
@@
 			)
 		)
-		(property "LCSC Part #" "C473237"
+		(property "LCSC Part #" "C863790"
 			(at 90.17 95.25 0)
 			(effects
@@
 		)
 		(property "Source" "LCSC"
+			(at 90.17 95.25 0)
+			(effects
+				(font
+					(size 1.27 1.27)
+				)
+				(hide yes)
+			)
+		)
+		(property "Alt" "ERA-3AEB392V"
+			(at 90.17 95.25 0)
+			(effects
+				(font
+					(size 1.27 1.27)
+				)
+				(hide yes)
+			)
+		)
+		(property "TME Part #" "-"
 			(at 90.17 95.25 0)
 			(effects
@@
 			)
 		)
-		(property "Footprint" "library:RT0603BRD0747KL"
+		(property "Footprint" "library:RT0603FRD0747KL"
 			(at 90.17 82.55 0)
 			(effects
@@
 			)
 		)
-		(property "LCSC Part #" "C326725"
+		(property "LCSC Part #" "C728633"
 			(at 90.17 82.55 0)
 			(effects
@@
 			)
 		)
-		(property "Mfr Part #" "RT0603BRD0747KL"
+		(property "Mfr Part #" "RT0603FRD0747KL"
 			(at 90.17 82.55 0)
 			(effects
@@
 			)
 		)
-		(property "Mouser Part #" "603-RT0603BRD0747KL"
+		(property "Mouser Part #" "603-RT0603FRD0747KL "
 			(at 90.17 82.55 0)
 			(effects
@@
 		)
 		(property "Source" "LCSC"
+			(at 90.17 82.55 0)
+			(effects
+				(font
+					(size 1.27 1.27)
+				)
+				(hide yes)
+			)
+		)
+		(property "Alt" "RT0603BRD0747KL"
+			(at 90.17 82.55 0)
+			(effects
+				(font
+					(size 1.27 1.27)
+				)
+				(hide yes)
+			)
+		)
+		(property "TME Part #" "-"
 			(at 90.17 82.55 0)
 			(effects
@@
 			)
 		)
-		(property "Footprint" "library:RT0603BRD0747KL"
+		(property "Footprint" "library:RT0603FRD0747KL"
 			(at 185.42 73.66 0)
 			(effects
@@
 			)
 		)
-		(property "LCSC Part #" "C326725"
+		(property "LCSC Part #" "C728633"
 			(at 185.42 73.66 0)
 			(effects
@@
 			)
 		)
-		(property "Mfr Part #" "RT0603BRD0747KL"
+		(property "Mfr Part #" "RT0603FRD0747KL"
 			(at 185.42 73.66 0)
 			(effects
@@
 			)
 		)
-		(property "Mouser Part #" "603-RT0603BRD0747KL"
+		(property "Mouser Part #" "603-RT0603FRD0747KL "
 			(at 185.42 73.66 0)
 			(effects
@@
 		)
 		(property "Source" "LCSC"
+			(at 185.42 73.66 0)
+			(effects
+				(font
+					(size 1.27 1.27)
+				)
+				(hide yes)
+			)
+		)
+		(property "Alt" "RT0603BRD0747KL"
+			(at 185.42 73.66 0)
+			(effects
+				(font
+					(size 1.27 1.27)
+				)
+				(hide yes)
+			)
+		)
+		(property "TME Part #" "-"
 			(at 185.42 73.66 0)
 			(effects
@@
 			(at 66.04 151.13 0)
 			(effects
+				(font
+					(size 1.27 1.27)
+				)
+				(hide yes)
+			)
+		)
+		(property "Alt" "OS102011MA1QN1C, OS102011MA1QS1, OS102011MA1QS1C, 1825232-1"
+			(at 66.04 151.13 0)
+			(effects

Commit message: schematic, PCB: many small adjustments before fab&assembly
Parts:
- RV301: JLCPCB Rotation Offset (none) -> -90
